File: kicad/_autosave-modular_ps.kicad_pcb (KiCad board)
At the start: 2 copper layers, 21 parts, among them J1 PJ-102AH, U1 LM7812_TO220, U2 LM7912_TO220

Commit message: schematic finished
Parts:
- added J2: Conn_01x01_Male, Connector_Pin:Pin_D1.3mm_L11.0mm, F.Cu at (55.9, 62.2)
Changed lines of the file:
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@@
     (tracks 0)
     (zones 0)
-    (modules 21)
+    (modules 22)
     (nets 7)
   )
@@
       (at (xyz 0 0 0))
       (scale (xyz 1 1 1))
+      (rotate (xyz 0 0 0))
+    )
+  )
+  (module Connector_Pin:Pin_D1.3mm_L11.0mm (layer F.Cu)
+    (at 55.88 62.23)
+    (descr "solder Pin_ diameter 1.3mm, hole diameter 1.3mm, length 11.0mm")
+    (tags "solder Pin_ pressfit")
+    (fp_text reference J2 (at 0 2.4) (layer F.SilkS)
+      (effects (font (size 1 1) (thickness 0.15)))
+    )
+    (fp_text value Conn_01x01_Male (at 0 -2.05) (layer F.Fab)
+      (effects (font (size 1 1) (thickness 0.15)))
+    )
+    (fp_circle (center 0 0) (end 1.6 0.05) (layer F.SilkS) (width 0.12))
+    (fp_circle (center 0 0) (end 1.25 -0.05) (layer F.Fab) (width 0.12))
+    (fp_circle (center 0 0) (end 0.65 -0.05) (layer F.Fab) (width 0.12))
+    (fp_circle (center 0 0) (end 1.8 0) (layer F.CrtYd) (width 0.05))
+    (fp_text user %R (at 0 2.4) (layer F.Fab)
+      (effects (font (size 1 1) (thickness 0.15)))
+    )
+    (pad 1 thru_hole circle (at 0 0) (size 2.6 2.6) (drill 1.3) (layers *.Cu *.Mask)
+      (net 4 +12V))
+    (model ${KISYS3DMOD}/Connector_Pin.3dshapes/Pin_D1.3mm_L11.0mm.wrl
+      (at (xyz 0 0 0))
+      (scale (xyz 1 1 1))
