File: kicad/modular_ps.sch (KiCad schematic (older format))
At the start: 21 parts, among them J1 PJ-102AH, U1 LM7912_TO220, U2 LM7812_TO220

Commit message: schematic finished
Parts:
- added +12V1: +12V, Connector_Pin:Pin_D1.3mm_L11.0mm, symbol Connector:Conn_01x01_Male
- added -12V1: -12V, Connector_Pin:Pin_D1.3mm_L11.0mm, symbol Connector:Conn_01x01_Male
- added GND1, GND? (x3): GND, Connector_Pin:Pin_D1.3mm_L11.0mm, symbol Connector:Conn_01x01_Male
- C10: renamed from C9; value CP1 -> 1uF; DIGI 478-1835-ND -> (none); DIGIKEY (none) -> 478-1835-ND
- C4: renamed from C7; value CP1 -> 1uF; DIGI 478-1835-ND -> (none); DIGIKEY (none) -> 478-1835-ND
- C5: renamed from C10; value CP1 -> 1uF; DIGI 478-1835-ND -> (none); DIGIKEY (none) -> 478-1835-ND
- C9: renamed from C8; value CP1 -> 1uF; DIGI 478-1835-ND -> (none); DIGIKEY (none) -> 478-1835-ND
- renumbered C3 to C2, C6 to C3, C2 to C6, C4 to C7, C5 to C8, D4 to D1, D1 to D2, D6 to D3, D3 to D4, D2 to D5, D5 to D6, U2 to U1, U1 to U2
Connections:
- net +12V: now also +12V1.1 (Pin_1)
- net -12V: now also -12V1.1 (Pin_1)
- net GND: now also GND1.1 (Pin_1), GND?.1 (Pin_1), GND?.1 (Pin_1), GND?.1 (Pin_1)
Other:
- moved on the sheet: C1, C10, C2, C3, C4, C5, C6, C7, C8, C9, D1, D2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

Commit message: commit for V1
Parts:
- removed +12V1: +12V, Connector_Pin:Pin_D1.3mm_L11.0mm, symbol Connector:Conn_01x01_Male
- removed -12V1: -12V, Connector_Pin:Pin_D1.3mm_L11.0mm, symbol Connector:Conn_01x01_Male
- removed D1, D2, D3, D4, D5, D6: 1N4004, Diode_THT:D_DO-41_SOD81_P10.16mm_Horizontal, symbol Diode:1N4004
- removed GND1, GND? (x3): GND, Connector_Pin:Pin_D1.3mm_L11.0mm, symbol Connector:Conn_01x01_Male
- removed R1, R2: 2.4K, Resistor_THT:R_Axial_DIN0207_L6.3mm_D2.5mm_P10.16mm_Horizontal, symbol Device:R
- removed U1: LM7812_TO220, Package_TO_SOT_THT:TO-220-3_Vertical, symbol Regulator_Linear:LM7812_TO220
- removed U2: LM7912_TO220, Package_TO_SOT_THT:TO-220-3_Vertical, symbol Regulator_Linear:LM7912_TO220
- added D1, D2, D3, D4, D5, D6: SM4004PL-TP, Diode_SMD:D_SOD-123F, symbol Diode:SM4004
- added J2: Conn_02x05_Counter_Clockwise, Connector_PinHeader_2.54mm:PinHeader_2x05_P2.54mm_Vertical, symbol Connector_Generic:Conn_02x05_Counter_Clockwise
- added U1: LM7812S/NOPB, Package_TO_SOT_SMD:TO-263-3_TabPin2, symbol Regulator_Linear:L7812
- added U2: LM2990SX-12/NOPB, Package_TO_SOT_SMD:TO-263-3_TabPin2, symbol Regulator_Linear:LM2990SX-12
Connections:
- net +12V: now also D1.2 (A), D3.1 (K), J2.1 (Pin_1), J2.2 (Pin_2), U1.3 (OUT)
- net -12V: now also D4.1 (K), D6.2 (A), J2.10 (Pin_10), J2.9 (Pin_9), U2.3 (OUT)
- net GND: now also D3.2 (A), D6.1 (K), J2.3 (Pin_3), J2.4 (Pin_4), J2.5 (Pin_5), J2.6 (Pin_6), J2.7 (Pin_7), J2.8 (Pin_8), U1.2 (GND), U2.1 (GND)
- net at C1.1, C2.1, C3.1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: now also D1.1 (K), D2.1 (K), U1.1 (IN)
- net at C6.2, C7.2, C8.2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: now also D4.2 (A), D5.2 (A), U2.2 (IN)
- net at J1.1: now also D2.2 (A), D5.1 (K)
